File: koyomi-keyboard-adapter.kicad_pcb (KiCad board)
At the start: 2 copper layers, 49.7 x 28.8 mm, 35 parts, among them J1 AXK750147G_VAIO-P, J2 BOOTSEL, J3 RUN, J4 USB, J5 BREAKOUT, J6 SWD, U1 RP2040, U2 AP2112K-3.3, U3 W25Q128JVS, Y1 ABM8-272-T3

Commit message: Changed PCB art to simple silkscreen lines
Parts:
- REF**: footprint exentio_art:exentio_blob_nocopper -> exentio_art:exentio_blob

Commit message: Decompressed matrix, broken out scroll lock LED, readme update
Parts:
- J5: footprint Connector_PinHeader_2.54mm:PinHeader_2x04_P2.54mm_Vertical -> Connector_PinHeader_2.54mm:PinHeader_2x05_P2.54mm_Vertical
- moved J5 2.54 mm to (24.2, 15.9)
Connections:
- J1 pad 1: COL13 -> COL14
- J1 pad 2: COL13 -> COL12
- J1 pad 24: COL14 -> COL15
- J1 pad 3: COL12 -> COL13
- J5 pad 1: SW_LID -> GND
- J5 pad 2: SW_PWR -> LED_SCRL
- J5 pad 3: LED_STBY -> SW_LID
- J5 pad 4: LED_WIFI -> SW_PWR
- J5 pad 5: LED_DISK -> LED_STBY
- J5 pad 6: SW_WIFI -> LED_WIFI
- J5 pad 7: LED_CHG -> LED_DISK
- J5 pad 8: LED_PWR -> SW_WIFI
- U1 pad 15: LED_SCRL -> COL14
- U1 pad 2: COL13 -> COL12
- U1 pad 3: COL12 -> COL13
- U1 pad 30: COL14 -> COL15
Routing:
- net COL15: track 0.00 -> 41.7 mm, vias 0 -> 2
- net COL14: track 41.3 -> 23.0 mm
- net COL13: track 22.9 -> 15.6 mm
- net COL12: track 15.6 -> 22.7 mm
- net SW_LID: track 30.8 -> 24.1 mm
- net LED_SCRL: track 16.8 -> 14.2 mm, vias 0 -> 1
- net SW_PWR: track 23.2 -> 20.6 mm
- net LED_STBY: track 27.6 -> 29.2 mm
- net ROW4: track 42.1 -> 42.8 mm
- net ROW7: track 49.2 -> 49.8 mm
- net ROW0: track 45.6 -> 46.3 mm
- net PS2_CLK: track 29.7 -> 30.3 mm
- net COL8: track 45.6 -> 46.1 mm
- net GND: vias 44 -> 66
Other:
- board text added: "1 3 5 7 9"
- board text added: "1 GND 2 LED_SCRLK 3 #SW_LID 4 #SW_PWR 5 LED_STBY 6 LED_WIFI 7 LED_DISK 8 SW_WIFI 9 LED_CHG 10 LED_PWR"
- board text added: "2 4 6 8 10"
- board text removed: "1 #SW_LID 2 #SW_PWR 3 LED_STBY 4 LED_WIFI 5 LED_DISK 6 SW_WIFI 7 LED_CHG 8 LED_PWR"
- board text removed: "1 3 5 7"
- board text removed: "2 4 6 8"
